Commit message: 🐛 fix(kuka_experimental): fix dimension

File: kuka_kr6_wsg_50_support/urdf/kr6r900sixx_macro.xacro (robot description, xacro)
@@ -113,5 +113,5 @@
         <link name="${prefix}tool0">
             <visual>
-                <origin xyz="0.0 -0.032 0.006" rpy="0 0 0"/>
+                <origin xyz="0.0 -0.032 0.0" rpy="0 0 0"/>
                 <geometry>
                     <mesh filename="package://wsg_50_simulation/meshes/WSG50_110.stl" scale="1 1 1"/>
@@ -123,5 +123,5 @@
             </visual>
             <collision>
-                <origin xyz="0.0 -0.032 0.006" rpy="0 0 0"/>
+                <origin xyz="0.0 -0.032 0.0" rpy="0 0 0"/>
                 <geometry>
                     <!--box size="0.146 0.05 0.0735"/-->
@@ -132,5 +132,5 @@
         <link name="wsg_50_gripper_left">
             <visual>
-                <origin xyz="0.0 -0.032 0.006" rpy="0 0 0"/>
+                <origin xyz="0.0 -0.032 0.0" rpy="0 0 0"/>
                 <geometry>
                     <mesh filename="package://wsg_50_simulation/meshes/GUIDE_WSG50_110.stl" scale="0.001 0.001 0.001"/>
@@ -142,5 +142,5 @@
             </visual>
             <collision>
-                <origin xyz="0 -0.032 0.006" rpy="0 0 0"/>
+                <origin xyz="0 -0.032 0.0" rpy="0 0 0"/>
                 <geometry>
                     <!--box size="0.0175 0.03 0.024"/-->
@@ -151,5 +151,5 @@
         <link name="wsg_50_finger_left">
             <visual>
-                <origin xyz="0.0 -0.032 0.006" rpy="0 0 0"/>
+                <origin xyz="0.0 -0.032 0.0" rpy="0 0 0"/>
                 <geometry>
                     <mesh filename="package://wsg_50_simulation/meshes/WSG-FMF.stl" scale="0.001 0.001 0.001"/>
@@ -160,5 +160,5 @@
             </visual>
             <collision>
-                <origin xyz="0 -0.032 0.006" rpy="0 0 0"/>
+                <origin xyz="0 -0.032 0.0" rpy="0 0 0"/>
                 <geometry>
                     <mesh filename="package://wsg_50_simulation/meshes/WSG-FMF.stl" scale="0.001 0.001 0.001"/>
@@ -168,5 +168,5 @@
         <link name="wsg_50_gripper_right">
             <visual>
-                <origin xyz="0.0 0.032 0.006" rpy="0 0 0"/>
+                <origin xyz="0.0 0.032 0.0" rpy="0 0 0"/>
                 <geometry>
                     <mesh filename="package://wsg_50_simulation/meshes/GUIDE_WSG50_110.stl" scale="0.001 0.001 0.001"/>
@@ -178,5 +178,5 @@
             </visual>
             <collision>
-                <origin xyz="0 0.032 0.006" rpy="0 0 0"/>
+                <origin xyz="0 0.032 0.0" rpy="0 0 0"/>
                 <geometry>
                     <!--box size="0.0175 0.03 0.024"/-->
@@ -187,5 +187,5 @@
         <link name="wsg_50_finger_right">
             <visual>
-                <origin xyz="0.0 0.032 0.006" rpy="0 0 0"/>
+                <origin xyz="0.0 0.032 0.0" rpy="0 0 0"/>
                 <geometry>
                     <mesh filename="package://wsg_50_simulation/meshes/WSG-FMF.stl" scale="0.001 0.001 0.001"/>
@@ -196,5 +196,5 @@
             </visual>
             <collision>
-                <origin xyz="0 0.032 0.006" rpy="0 0 0"/>
+                <origin xyz="0 0.032 0.0" rpy="0 0 0"/>
                 <geometry>
                     <mesh filename="package://wsg_50_simulation/meshes/WSG-FMF.stl" scale="0.001 0.001 0.001"/>

Commit message: ✨ feat(kuka_experimental): add ground object

File: kuka_kr6_wsg_50_support/urdf/kr6r900sixx_macro.xacro (robot description, xacro)
@@ -202,4 +202,26 @@
             </collision>
         </link>
+        <link name="ground_plane_box">
+            <visual>
+                <origin xyz="0 0 0" rpy="0 0 0"/>
+                <geometry>
+                    <box size="2.0 2.0 0.01"/>
+                </geometry>
+                <material name="Grey">
+                    <color rgba="0 0 0 1.0"/>
+                </material>
+            </visual>
+            <collision>
+                <origin xyz="0 0 0" rpy="0 0 0"/>
+                <geometry>
+                    <box size="2.0 2.0 0.01"/>
+                </geometry>
+            </collision>
+        </link>
+        <joint name="ground_plane_box" type="fixed">
+            <parent link="base_link"/>
+            <child link="ground_plane_box"/>
+            <origin xyz="0 0 0" rpy="0 0 0"/>
+        </joint>
         <link name="wsg_50_joint_finger_center">
         </link>
